Commit message: setup xacro and launch file

File: description/robot_core.xacro (robot description, xacro)
@@ -1,3 +1,11 @@
 <?xml version="1.0"?>
 <robot xmlns:xacro="http://www.ros.org/wiki/xacro">
+    <link name="base_link">
+        <visual>
+            <geometry>
+                <box size="1 1 1" />
+                <origin xyz="0 0 0" rpy="0 0 0" />
+            </geometry>
+        </visual>
+    </link>
 </robot>

Commit message: adds robot_core xacro

File: description/robot_core.xacro (robot description, xacro)
@@ -1,10 +1,30 @@
 <?xml version="1.0"?>
 <robot xmlns:xacro="http://www.ros.org/wiki/xacro">
+    <material name="white">
+        <color rgba="1 1 1 1"/>
+    </material>
+    <material name="orange">
+        <color rgba="1 0.3 0.1 1"/>
+    </material>
+    <material name="blue">
+        <color rgba="0.2 0.2 1 1"/>
+    </material>
+    <material name="black">
+        <color rgba="0 0 0 1"/>
+    </material>
     <link name="base_link">
+    </link>
+    <joint name="chassis_joint" type="fixed">
+        <parent link="base_link"/>
+        <child link="chassis"/>
+        <origin xyz="-0.1 0 0"/>
+    </joint>
+    <link name="chassis">
         <visual>
+            <origin xyz="0.15 0 0.075"/>
             <geometry>
-                <box size="1 1 1" />
-                <origin xyz="0 0 0" rpy="0 0 0" />
+                <box size="0.3 0.3 0.15"/>
             </geometry>
+            <material name="white"/>
         </visual>
     </link>

Commit message: xacro setup completed

File: description/robot_core.xacro (robot description, xacro)
@@ -13,6 +13,8 @@
         <color rgba="0 0 0 1"/>
     </material>
+    <!-- BASE LINK -->
     <link name="base_link">
     </link>
+    <!-- CHASSIS LINK -->
     <joint name="chassis_joint" type="fixed">
         <parent link="base_link"/>
@@ -26,5 +28,63 @@
                 <box size="0.3 0.3 0.15"/>
             </geometry>
-            <material name="white"/>
+            <material name="black"/>
+        </visual>
+    </link>
+    <!-- LEFT WHEEL LINK -->
+    <joint name="left_wheel_joint" type="continuous">
+        <parent link="base_link"/>
+        <child link="left_wheel"/>
+        <origin xyz="0 0.175 0" rpy="-${pi/2} 0 0"/>
+        <axis xyz="0 0 1"/>
+    </joint>
+    <link name="left_wheel">
+        <visual>
+            <geometry>
+                <cylinder length="0.04" radius="0.05"/>
+            </geometry>
+            <material name="blue"/>
+        </visual>
+    </link>
+    <!-- RIGHT WHEEL LINK -->
+    <joint name="right_wheel_joint" type="continuous">
+        <parent link="base_link"/>
+        <child link="right_wheel"/>
+        <origin xyz="0 -0.175 0" rpy="${pi/2} 0 0"/>
+        <axis xyz="0 0 1"/>
+    </joint>
+    <link name="right_wheel">
+        <visual>
+            <geometry>
+                <cylinder length="0.04" radius="0.05"/>
+            </geometry>
+            <material name="blue"/>
+        </visual>
+    </link>
+    <!-- CASTER WHEEL LINK -->
+    <joint name="caster_wheel_joint" type="fixed">
+        <parent link="chassis"/>
+        <child link="caster_wheel"/>
+        <origin xyz="0.24 0 0"/>
+    </joint>
+    <link name="caster_wheel">
+        <visual>
+            <geometry>
+                <sphere radius="0.05"/>
+            </geometry>
+            <material name="blue"/>
+        </visual>
+    </link>
+    <!-- LIDAR LINK -->
+    <joint name="laser_frame_joint" type="fixed">
+        <parent link="base_link"/>
+        <child link="laser_frame"/>
+        <origin xyz="0 0 0.175"/>
+    </joint>
+    <link name="laser_frame">
+        <visual>
+            <geometry>
+                <cylinder length="0.04" radius="0.05"/>
+            </geometry>
+            <material name="orange"/>
         </visual>
     </link>

Commit message: lidar urdf aligned

File: description/robot_core.xacro (robot description, xacro)
@@ -79,5 +79,6 @@
         <parent link="base_link"/>
         <child link="laser_frame"/>
-        <origin xyz="0 0 0.175"/>
+        <origin xyz="0 0 0.175" rpy="${pi} 0 0"/>
+        <axis xyz="0 0 1"/>
     </joint>
     <link name="laser_frame">

Commit message: odometry setup with errors

File: description/robot_core.xacro (robot description, xacro)
@@ -32,5 +32,6 @@
     </link>
     <!-- LEFT WHEEL LINK -->
-    <joint name="left_wheel_joint" type="continuous">
+    <!-- <joint name="left_wheel_joint" type="continuous"> -->
+    <joint name="left_wheel_joint" type="fixed">
         <parent link="base_link"/>
         <child link="left_wheel"/>
@@ -47,5 +48,6 @@
     </link>
     <!-- RIGHT WHEEL LINK -->
-    <joint name="right_wheel_joint" type="continuous">
+    <!-- <joint name="right_wheel_joint" type="continuous"> -->
+    <joint name="right_wheel_joint" type="fixed">
         <parent link="base_link"/>
         <child link="right_wheel"/>

Commit message: il commit più inutile della storia

File: description/robot_core.xacro (robot description, xacro)
@@ -20,11 +20,20 @@
         <parent link="base_link"/>
         <child link="chassis"/>
-        <origin xyz="-0.1 0 0"/>
+        <origin xyz="-0.15 0 0"/>
     </joint>
-    <link name="chassis">
+    <!-- <link name="chassis">
         <visual>
             <origin xyz="0.15 0 0.075"/>
             <geometry>
                 <box size="0.3 0.3 0.15"/>
+            </geometry>
+            <material name="black"/>
+        </visual>
+    </link> -->
+        <link name="chassis">
+        <visual>
+            <origin xyz="0.15 0 0.075"/>
+            <geometry>
+                <cylinder length="0.10" radius="0.15"/>
             </geometry>
             <material name="black"/>
@@ -42,5 +51,5 @@
         <visual>
             <geometry>
-                <cylinder length="0.04" radius="0.05"/>
+                <cylinder length="0.04" radius="0.04"/>
             </geometry>
             <material name="blue"/>
@@ -58,5 +67,5 @@
         <visual>
             <geometry>
-                <cylinder length="0.04" radius="0.05"/>
+                <cylinder length="0.04" radius="0.04"/>
             </geometry>
             <material name="blue"/>
@@ -64,5 +73,5 @@
     </link>
     <!-- CASTER WHEEL LINK -->
-    <joint name="caster_wheel_joint" type="fixed">
+    <!-- <joint name="caster_wheel_joint" type="fixed">
         <parent link="chassis"/>
         <child link="caster_wheel"/>
@@ -76,5 +85,5 @@
             <material name="blue"/>
         </visual>
-    </link>
+    </link> -->
     <!-- LIDAR LINK -->
     <joint name="laser_frame_joint" type="fixed">

Commit message: unified sensor and actuator control and publication of topic on the robot side, cleaned derectory from old code, update readme.md.

File: description/robot_core.xacro (robot description, xacro)
@@ -22,14 +22,5 @@
         <origin xyz="-0.15 0 0"/>
     </joint>
-    <!-- <link name="chassis">
-        <visual>
-            <origin xyz="0.15 0 0.075"/>
-            <geometry>
-                <box size="0.3 0.3 0.15"/>
-            </geometry>
-            <material name="black"/>
-        </visual>
-    </link> -->
-        <link name="chassis">
+    <link name="chassis">
         <visual>
             <origin xyz="0.15 0 0.075"/>

Commit message: Update README.md

File: description/robot_core.xacro (robot description, xacro)
@@ -42,5 +42,5 @@
         <visual>
             <geometry>
-                <cylinder length="0.04" radius="0.04"/>
+                <cylinder length="0.035" radius="0.065"/>
             </geometry>
             <material name="blue"/>
@@ -58,5 +58,5 @@
         <visual>
             <geometry>
-                <cylinder length="0.04" radius="0.04"/>
+                <cylinder length="0.035" radius="0.065"/>
             </geometry>
             <material name="blue"/>
